Commit message: Added M_PI definition

File: urdf/kinect.urdf.xacro (robot description, xacro)
@@ -13,5 +13,7 @@
     xmlns:physics="http://playerstage.sourceforge.net/gazebo/xmlschema/#physics"
     xmlns:xacro="http://ros.org/wiki/xacro">
-<xacro:macro name="kinect" params="xyz rpy parent_frame" >
+  <!-- math constants -->
+  <xacro:property name="M_PI" value="3.1415926535897931" />
+  <xacro:macro name="kinect" params="xyz rpy parent_frame" >
   <joint name="base_camera_joint" type="fixed">
     <origin xyz="${xyz}" rpy="${rpy}" />

Commit message: ROS2-Humble port

File: urdf/kinect.urdf.xacro (robot description, xacro)
@@ -1,4 +1,4 @@
 <?xml version="1.0"?>
-<robot xmlns:xi="http://www.w3.org/2001/XInclude"
+<robot name="ur"
     xmlns:gazebo="http://playerstage.sourceforge.net/gazebo/xmlschema/#gz"
     xmlns:model="http://playerstage.sourceforge.net/gazebo/xmlschema/#model"
@@ -13,90 +13,12 @@
     xmlns:physics="http://playerstage.sourceforge.net/gazebo/xmlschema/#physics"
     xmlns:xacro="http://ros.org/wiki/xacro">
-  <!-- math constants -->
-  <xacro:property name="M_PI" value="3.1415926535897931" />
-  <xacro:macro name="kinect" params="xyz rpy parent_frame" >
-  <joint name="base_camera_joint" type="fixed">
-    <origin xyz="${xyz}" rpy="${rpy}" />
-    <parent link="${parent_frame}" />
-    <origin xyz="0 0 0" rpy="0 0 0" />
-    <child link="camera_link" />
-  </joint>
-  <link name="camera_link">
-    <inertial>
-      <mass value="0.01" />
-      <origin xyz="0 0 0" />
-      <inertia ixx="0.001" ixy="0.0" ixz="0.0"
-        iyy="0.001" iyz="0.0"
-        izz="0.001" />
-    </inertial>
-    <visual>
-      <origin xyz=" 0 0 0 " rpy="0 0 0" />
-      <geometry>
-        <mesh filename="package://kinect_description/meshes/kinect.dae"/>
-      </geometry>
-    </visual>
-    <collision>
-      <origin xyz="0.0 0.0 0.0" rpy="0 0 0" />
-      <geometry>
-        <box size="0.0730 .2760 0.0720"/>
-      </geometry>
-    </collision>
-  </link>
-  <joint name="camera_depth_joint" type="fixed">
-    <origin xyz="0 0.011 0" rpy="0 0 0" />
-    <parent link="camera_link" />
-    <child link="camera_depth_frame" />
-  </joint>
-  <link name="camera_depth_frame">
-    <inertial>
-      <mass value="0.01" />
-      <origin xyz="0 0 0" />
-      <inertia ixx="0.001" ixy="0.0" ixz="0.0"
-        iyy="0.001" iyz="0.0"
-        izz="0.001" />
-    </inertial>
-  </link>
-  <joint name="camera_depth_optical_joint" type="fixed">
-    <origin xyz="0 0 0" rpy="${-M_PI/2} 0 ${-M_PI/2}" />
-    <parent link="camera_depth_frame" />
-    <child link="camera_depth_optical_frame" />
-  </joint>
-  <link name="camera_depth_optical_frame">
-    <inertial>
-      <mass value="0.001" />
-      <origin xyz="0 0 0" />
-      <inertia ixx="0.0001" ixy="0.0" ixz="0.0"
-        iyy="0.0001" iyz="0.0"
-        izz="0.0001" />
-    </inertial>
-  </link>
-  <joint name="camera_rgb_joint" type="fixed">
-    <origin xyz="0 -0.012 0" rpy="0 0 0" />
-    <parent link="camera_link" />
-    <child link="camera_rgb_frame" />
-  </joint>
-  <link name="camera_rgb_frame">
-    <inertial>
-      <mass value="0.001" />
-      <origin xyz="0 0 0" />
-      <inertia ixx="0.0001" ixy="0.0" ixz="0.0"
-        iyy="0.0001" iyz="0.0"
-        izz="0.0001" />
-    </inertial>
-  </link>
-  <joint name="camera_rgb_optical_joint" type="fixed">
-    <origin xyz="0 0 0" rpy="${-M_PI/2} 0 ${-M_PI/2}" />
-    <parent link="camera_rgb_frame" />
-    <child link="camera_rgb_optical_frame" />
-  </joint>
-  <link name="camera_rgb_optical_frame">
-    <inertial>
-      <mass value="0.001" />
-      <origin xyz="0 0 0" />
-      <inertia ixx="0.0001" ixy="0.0" ixz="0.0"
-        iyy="0.0001" iyz="0.0"
-        izz="0.0001" />
-    </inertial>
-  </link>
-</xacro:macro>
+    <xacro:arg name="prefix" default=""/>
+    <!-- Kinect model -->
+	<xacro:include filename="$(find kinect_description)/urdf/kinect_macro.xacro"/>
+	<link name="base_link"/>
+	<xacro:kinect
+		xyz="0.0 0.0 0.0"
+		rpy="0.0 0.0 0.0"
+		parent_frame="base_link"
+		prefix="$(arg prefix)"/>
 </robot>
